Commit message: robotic_arm project updated

File: ros_portfolio/robotic_arm/ros_ws/src/robotic_arm/description/arm.urdf.xacro (robot description, xacro)
@@ -1,4 +1,6 @@
 <?xml version="1.0"?>
 <robot xmlns:xacro="http://www.ros.org/wiki/xacro" name="robotic_arm">
+    <xacro:include filename="$(find robotic_arm)/description/arm_gazebo.urdf.xacro"/>
+    <xacro:include filename="$(find robotic_arm)/description/arm_control.urdf.xacro"/>
     <xacro:property name="PI" value="3.14159265359" />
     <xacro:property name="effort" value="30.0" />
@@ -12,4 +14,13 @@
                      izz="1.0" />
         </inertial>
+    </xacro:macro>
+    <xacro:macro name="default_transmission" params="number">
+        <transmission name="transmission_${number}">
+            <type>transmission_interface/SimpleTransmission</type>
+            <actuator name="motor_${number}" role="actuator1"/>
+            <joint name="joint_${number}" role="joint1">
+                <mechanicalReduction>1.0</mechanicalReduction>
+            </joint>
+        </transmission>
     </xacro:macro>
     <link name="world"/>
@@ -170,3 +181,7 @@
         <mimic joint="joint_4" multiplier="-1"/>
     </joint>
+    <xacro:default_transmission number="1"/>
+    <xacro:default_transmission number="2"/>
+    <xacro:default_transmission number="3"/>
+    <xacro:default_transmission number="4"/>
 </robot>
